File: pcb/MacPicoModem.kicad_pcb (KiCad board)
At the start: 2 copper layers, 67.6 x 128.2 mm, 22 parts, among them J1 DIN-802, J2 TYPE-C 16PIN 2MD, SW1 K2-1102AQ-J4CW-01, U1 SP3238EEA-L/TR, U2 74HCT245, U3 Pico, U4 24LC32A-I/SN

Commit message: launch
Parts:
- added R6: 0805W8F5101T5E, EasyEDA:R0805, F.Cu at (132.0, 50.7)
- added R7: 0805W8F5101T5E, EasyEDA:R0805, F.Cu at (132.0, 46.7)
Connections:
- J1 pad 4: GND -> Net-(U1-T1OUT)
- J1 pad 5: Net-(U1-T1OUT) -> unconnected-(J1-Pad5)
- J1 pad 6: unconnected-(J1-Pad6) -> GND
- J2 pad A4B9: unconnected-(J2-VBUS-PadA4B9) -> +5V
- J2 pad A5: unconnected-(J2-CC1-PadA5) -> Net-(J2-CC1)
- J2 pad B5: unconnected-(J2-CC2-PadB5) -> Net-(J2-CC2)
- J2 pad B6: unconnected-(J2-Dp2-PadB6) -> Net-(J2-Dp1)
- J2 pad B7: unconnected-(J2-Dn2-PadB7) -> Net-(J2-Dn1)
- U2 pad 12: Net-(D3-A) -> unconnected-(U2-B6-Pad12)
- U2 pad 13: unconnected-(U2-B5-Pad13) -> Net-(D3-A)
Routing:
- net Net-(J2-CC1): track 0.00 -> 12.0 mm
- net Net-(J2-CC2): track 0.00 -> 11.8 mm, vias 0 -> 2
- net +5V: track 242.5 -> 250.4 mm
- net Net-(U1-T1OUT): track 33.6 -> 39.3 mm, vias 2 -> 0
- net Net-(J2-Dp1): track 36.4 -> 41.6 mm
- net Net-(J2-Dn1): track 34.2 -> 38.4 mm, vias 0 -> 2
- net Net-(U1-R1IN): track 37.4 -> 36.0 mm
- net GND: track 40.6 -> 40.2 mm, vias 45 -> 48
