File: pcb/MacPicoModem.kicad_sch (KiCad schematic)
At the start: 32 parts, among them J1 Mini-DIN-8, P1 CONN_02X05, P2 USB_C_Plug_USB2.0, SW1 SW_SPST, U1 MAX3237CAI+, U2 74HCT245, U3 Pico, U5 24LC32

Commit message: first pcb and case
Parts:
- removed D1, D2, D3, D4, D5, D6, D7, D8: TLPR5600, modules:LED-3MM, symbol Pico_Wifi_modem:LED
- removed J1: Mini-DIN-8, symbol Connector:Mini-DIN-8
- removed P1: CONN_02X05, modules:IDC_Header_Straight_10pins, symbol Pico_Wifi_modem:CONN_02X05
- removed P2: USB_C_Plug_USB2.0, symbol Connector:USB_C_Plug_USB2.0
- removed R1, R2, R5, R6, R8: 560R, modules:R3, symbol Pico_Wifi_modem:R_US
- removed SW1: SW_SPST, symbol Switch:SW_SPST
- removed U1: MAX3237CAI+, modules:SOIC-28W_7.5x17.9mm_Pitch1.27mm, symbol Pico_Wifi_modem:MAX3237CAI+
- removed U5: 24LC32, modules:DIP-8_W7.62mm_LongPads, symbol Pico_Wifi_modem:24LC32
- added C7: 100nF, Capacitor_SMD:C_0805_2012Metric, symbol Pico_Wifi_modem:C_Small
- added D1, D2, D3: FC-2012UGK-520D5, EasyEDA:LED0805-R-RD, symbol EasyEDA:FC-2012UGK-520D5
- added J1: DIN-802, EasyEDA:CONN-TH_DIN-802, symbol EasyEDA:DIN-802
- added J2: TYPE-C 16PIN 2MD, EasyEDA:USB-C-SMD_TYPE-C-16PIN-2MD-073, symbol EasyEDA:TYPE-C16PIN2MD
- added SW1: K2-1102AQ-J4CW-01, EasyEDA:KEY-TH_K2-1102AQ-JXXW-XX, symbol EasyEDA:K2-1102AQ-J4CW-01
- added U1: SP3238EEA-L/TR, EasyEDA:SSOP-28_L10.2-W5.3-P0.65-LS7.8-BL, symbol EasyEDA:SP3238EEA-L_TR
- added U4: 24LC32A-I/SN, EasyEDA:SOIC-8_L4.9-W3.9-P1.27-LS6.0-BL, symbol EasyEDA:24LC32A-I_SN
- C1, C2, C3, C4, C5: footprint modules:C_Disc_D3_P2.5 -> Capacitor_SMD:C_0805_2012Metric; LCSC Part (none) -> C1711; Price 0.37 -> (none)
- C6: footprint modules:C_Disc_D3_P5 -> Capacitor_SMD:C_0805_2012Metric; LCSC Part (none) -> C1711; Price 0.34 -> (none)
- R1: renamed from R3; footprint modules:R3 -> Resistor_SMD:R_0805_2012Metric; LCSC Part (none) -> C114536; Price 0.16 -> (none)
- R2: renamed from R4; footprint modules:R3 -> Resistor_SMD:R_0805_2012Metric; LCSC Part (none) -> C114536; Price 0.16 -> (none)
- R3: renamed from R7; footprint modules:R3 -> Resistor_SMD:R_0805_2012Metric; LCSC Part (none) -> C114536; Price 0.16 -> (none)
- R4: renamed from R12; footprint modules:R3 -> Resistor_SMD:R_0805_2012Metric; LCSC Part (none) -> C2907252
- R5: renamed from R13; footprint modules:R3 -> Resistor_SMD:R_0805_2012Metric; LCSC Part (none) -> C2907252
- U2: footprint modules:DIP-20_W7.62mm_LongPads -> EasyEDA:TSSOP-20_L6.5-W4.4-P0.65-LS6.4-BL; LCSC Part (none) -> C52140501
- U3: footprint modules:RPi_PicoW -> Module:RaspberryPi_Pico_W_SMD
Connections:
- net +5V: now also C7.1, J2.B4A9 (VBUS), U1.14 (~{SHUTDOWN}), U1.26 (VCC), U4.8 (VCC)
- net GND: now also R1.2, R2.2, R3.2, C7.2, J1.4, J1.8, J2.A1B12 (GND), J2.B1A12 (GND), SW1.2, U1.13 (~{ONLINE}), U1.15 (~{STATUS}), U1.2 (GND), U4.1 (A0), U4.2 (A1), U4.3 (A2), U4.4 (VSS), U4.7 (WP)
- net at C1.1: now also U1.1 (C2+)
- net at C1.2: now also U1.3 (C2-)
- net at C6.1: now also U1.28 (C1+)
- net at C6.2: now also U1.25 (C1-)
- net at C2.1: now also U1.4 (V-)
- net at C3.2: now also U1.27 (V+)
- net at R3.1: now also D3.2 (K); no longer U2.12 (B6)
- net at R2.1: now also D2.2 (K); no longer U2.15 (B3)
- net at R1.1: now also D1.2 (K); no longer U2.16 (B2)
- net at U2.5 (A3), U3.1 (GPIO0): now also U1.24 (T1IN)
- net at U2.6 (A4), U3.10 (GPIO7): now also U1.17 (T5IN)
- net at U2.4 (A2), U3.2 (GPIO1): now also U1.21 (R1OUT)
- net at R5.2, U3.21 (GPIO16): now also U4.5 (SDA)
- net at R4.2, U3.22 (GPIO17): now also U4.6 (SCL)
- net at U2.9 (A7), U3.4 (GPIO2): now also U1.20 (R2OUT)
- net at U2.8 (A6), U3.5 (GPIO3): now also U1.23 (T2IN)
- net at U2.7 (A5), U3.6 (GPIO4): now also U1.22 (T3IN)
- net at U2.2 (A0), U3.7 (GPIO5): now also U1.19 (T4IN)
- net at U2.3 (A1), U3.9 (GPIO6): now also U1.18 (R3OUT)
- net at U3.TP2 (D-): now also J2.A7 (Dn1)
- net at U3.TP3 (D+): now also J2.A6 (Dp1)
- net at U3.TP6 (BOOTSEL): now also SW1.1
- new net: D3.1 (A), U2.12 (B6)
- new net: D2.1 (A), U2.15 (B3)
- new net: D1.1 (A), U2.16 (B2)
- new net: J1.1, U1.9 (R2IN)
- new net: J1.2, U1.6 (T2OUT)
- new net: J1.3, U1.8 (R1IN)
- new net: J1.5, U1.5 (T1OUT)
- no-connect marks 25 -> 23
Other:
- note removed: "CD"
- note removed: "CS"
- note removed: "MR"
- note removed: "RD"
- note removed: "RS"
- note removed: "RxD"
- note removed: "SD"
- note removed: "TR"
- note removed: "TxD"
- moved on the sheet: C2, C3, C5, C6, R1, R2, R3

Commit message: launch
Parts:
- added R6, R7: 0805W8F5101T5E, EasyEDA:R0805, symbol EasyEDA:0805W8F5101T5E
Connections:
- net +5V: now also J2.A4B9 (VBUS)
- net GND: now also J1.6, R6.2, R7.2; no longer J1.4
- net at J2.A7 (Dn1), U3.TP2 (D-): now also J2.B7 (Dn2)
- net at J2.A6 (Dp1), U3.TP3 (D+): now also J2.B6 (Dp2)
- net at U2.12 (B6): no longer D3.1 (A)
- net at U2.13 (B5): now also D3.1 (A)
- net at U1.5 (T1OUT): now also J1.4; no longer J1.5
- net at J2.A5 (CC1): now also R7.1
- net at J2.B5 (CC2): now also R6.1
- no-connect marks 23 -> 25
